File: RTI-Dome-Hardware/RTI-Dome.sch (EAGLE design)
At the start: 31 parts, among them IC2 74LVC244

Commit message: Fix small error on schematics
Other:
- note removed: "Pin 0 and 1 are connected to XBee"
Changed lines of the file:
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@@
 <sheet>
 <plain>
-<text x="129.54" y="35.56" size="1.016" layer="97">Pin 0 and 1 are connected to XBee</text>
 </plain>
 <instances>

Commit message: Stop interrupt in motor disable code.
Parts:
- added X11: (no value), con-ptr500:AK500/2
Connections:
- new net AT_PARK_PIN: PCB1.A5, X11-1.KL
- new net AT_PARK_PIN_LOOP: PCB1.A4, X11-2.KL
Changed lines of the file:
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@@
 <part name="R2" library="rti" deviceset="R-EU" device="'0805'" value="100K 0.1%"/>
 <part name="C3" library="rti" deviceset="C-EU" device="'0805'" value="10uF"/>
+<part name="X11" library="con-ptr500" deviceset="AK500/2" device=""/>
 </parts>
 <sheets>
@@
 <instance part="R2" gate="G$1" x="5.08" y="129.54" rot="R90"/>
 <instance part="C3" gate="G$1" x="185.42" y="53.34"/>
+<instance part="X11" gate="-1" x="48.26" y="27.94" rot="R180"/>
+<instance part="X11" gate="-2" x="48.26" y="33.02" rot="R180"/>
 </instances>
 <busses>
@@
 </segment>
 </net>
+<net name="AT_PARK_PIN_LOOP" class="0">
+<segment>
+<pinref part="X11" gate="-2" pin="KL"/>
+<wire x1="40.64" y1="33.02" x2="43.18" y2="33.02" width="0.1524" layer="91"/>
+<label x="40.64" y="33.02" size="1.016" layer="95" rot="R180" xref="yes"/>
+</segment>
+<segment>
+<wire x1="73.66" y1="43.18" x2="76.2" y2="43.18" width="0.1524" layer="91"/>
+<label x="73.66" y="43.18" size="1.016" layer="95" rot="R180" xref="yes"/>
+<pinref part="PCB1" gate="G$1" pin="A4"/>
+</segment>
+</net>
+<net name="AT_PARK_PIN" class="0">
+<segment>
+<pinref part="X11" gate="-1" pin="KL"/>
+<wire x1="40.64" y1="27.94" x2="43.18" y2="27.94" width="0.1524" layer="91"/>
+<label x="40.64" y="27.94" size="1.016" layer="95" rot="R180" xref="yes"/>
+</segment>
+<segment>
+<wire x1="73.66" y1="40.64" x2="76.2" y2="40.64" width="0.1524" layer="91"/>
+<label x="73.66" y="40.64" size="1.016" layer="95" rot="R180" xref="yes"/>
+<pinref part="PCB1" gate="G$1" pin="A5"/>
+</segment>
+</net>
