File: Hardware/RTI-Dome.brd (EAGLE design)
At the start: 80 x 71.1 mm, 50 parts, among them IC1 24AA128ST, IC2 MCP120T-270I_TT, IC3 FT232RL, IC5 74LVC245, IC6 74ABT245, X13 PN61729-S

Commit message: PCB optimisation
Parts:
- removed X12: (no value), con-ptr500:AK500/2
- moved X2 4.49 mm to (75.6, 18.4)
- moved C2 2.86 mm to (64.5, 18.1)
Connections:
- net GND: no longer X12.1, X12.2
Routing:
- net +12V: track 149.1 -> 143.0 mm
Changed lines of the file:
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@@
 </autorouter>
 <elements>
-<element name="X2" library="con-ptr500" package="AK500/2" value="" x="74.93" y="13.97" rot="R90">
-<attribute name="OC_FARNELL" value="unknown" x="74.93" y="13.97" size="1.778" layer="27" rot="R90" display="off"/>
-<attribute name="OC_NEWARK" value="unknown" x="74.93" y="13.97" size="1.778" layer="27" rot="R90" display="off"/>
-<attribute name="MF" value="" x="74.93" y="13.97" size="1.778" layer="27" rot="R90" display="off"/>
-<attribute name="MPN" value="" x="74.93" y="13.97" size="1.778" layer="27" rot="R90" display="off"/>
+<element name="X2" library="con-ptr500" package="AK500/2" value="" x="75.565" y="18.415" rot="R90">
+<attribute name="OC_FARNELL" value="unknown" x="75.565" y="18.415" size="1.778" layer="27" rot="R90" display="off"/>
+<attribute name="OC_NEWARK" value="unknown" x="75.565" y="18.415" size="1.778" layer="27" rot="R90" display="off"/>
+<attribute name="MF" value="" x="75.565" y="18.415" size="1.778" layer="27" rot="R90" display="off"/>
+<attribute name="MPN" value="" x="75.565" y="18.415" size="1.778" layer="27" rot="R90" display="off"/>
 </element>
 <element name="X4" library="con-ptr500" package="AK500/3" value="" x="53.84" y="65.7225" rot="R180">
@@
 <element name="R5" library="rti" package="R0805" value="100" x="33.02" y="54.61" rot="R90"/>
 <element name="U$4" library="rti" package="LOGO_BIG" value="RTI-LOGO_BIG" x="36.195" y="19.812"/>
-<element name="C2" library="rti" package="UD-10X10_NICHICON" value="100uF" x="64.4525" y="15.24" rot="R270"/>
+<element name="C2" library="rti" package="UD-10X10_NICHICON" value="100uF" x="64.4525" y="18.0975" rot="R270"/>
 <element name="R13" library="rti" package="R0805" value="4.7K" x="5.08" y="20.3835" rot="R180"/>
 <element name="R14" library="rti" package="R0805" value="4.7K" x="5.08" y="16.256"/>
@@
 <element name="R3" library="rti" package="R0805" value="1K" x="1.93675" y="44.45" rot="R270"/>
 <element name="C5" library="rti" package="C0805" value="100nF" x="1.93675" y="40.22725" rot="R270"/>
-<element name="X12" library="con-ptr500" package="AK500/2" value="" x="43.18" y="3.81">
-<attribute name="OC_NEWARK" value="unknown" x="43.18" y="3.81" size="1.778" layer="27" display="off"/>
-<attribute name="OC_FARNELL" value="unknown" x="43.18" y="3.81" size="1.778" layer="27" display="off"/>
-<attribute name="MF" value="" x="43.18" y="3.81" size="1.778" layer="27" display="off"/>
-<attribute name="MPN" value="" x="43.18" y="3.81" size="1.778" layer="27" display="off"/>
-</element>
 <element name="IC3" library="ftdichip" package="SSOP28" value="FT232RL" x="64.77" y="31.75">
 <attribute name="MF" value="" x="64.77" y="64.77" size="1.778" layer="27" display="off"/>
@@
 <contactref element="PCB1" pad="GND.."/>
 <contactref element="C3" pad="2"/>
-<via x="62.23" y="16.51" extent="1-16" drill="0.6" diameter="1.27"/>
+<via x="56.1975" y="25.0825" extent="1-16" drill="0.6" diameter="1.27"/>
 <contactref element="X7" pad="1"/>
 <contactref element="X8" pad="1"/>
@@
 <contactref element="C9" pad="2"/>
 <via x="62.23" y="39.37" extent="1-16" drill="0.6" diameter="1.27"/>
-<via x="60.96" y="20.32" extent="1-16" drill="0.6" diameter="1.27"/>
 <via x="50.8" y="17.78" extent="1-16" drill="0.6" diameter="1.27"/>
 <via x="34.29" y="21.59" extent="1-16" drill="0.6" diameter="1.27"/>
 <via x="54.61" y="33.02" extent="1-16" drill="0.6" diameter="1.27"/>
-<via x="64.4525" y="22.225" extent="1-16" drill="0.6" diameter="1.27"/>
-<via x="67.31" y="20.32" extent="1-16" drill="0.6" diameter="1.27"/>
-<via x="69.85" y="20.32" extent="1-16" drill="0.6" diameter="1.27"/>
-<via x="72.39" y="20.32" extent="1-16" drill="0.6" diameter="1.27"/>
+<via x="64.4525" y="25.4" extent="1-16" drill="0.6" diameter="1.27"/>
+<via x="56.8325" y="18.7325" extent="1-16" drill="0.6" diameter="1.27"/>
 <via x="43.18" y="54.61" extent="1-16" drill="0.6" diameter="1.27"/>
 <via x="34.95675" y="38.227" extent="1-16" drill="0.6" diameter="1.27"/>
@@
 <via x="3.81" y="34.29" extent="1-16" drill="0.6" diameter="1.27"/>
 <via x="31.75" y="34.29" extent="1-16" drill="0.6" diameter="1.27"/>
-<contactref element="X12" pad="1"/>
 <via x="66.04" y="31.75" extent="1-16" drill="0.6" diameter="1.27"/>
-<contactref element="X12" pad="2"/>
 <via x="11.43" y="24.13" extent="1-16" drill="0.6" diameter="1.27"/>
 <via x="13.97" y="12.7" extent="1-16" drill="0.6" diameter="1.27"/>
@@
 <via x="10.38225" y="15.90675" extent="1-16" drill="0.6" diameter="1.27"/>
 <via x="33.02" y="3.81" extent="1-16" drill="0.6" diameter="1.27"/>
-<via x="35.56" y="3.81" extent="1-16" drill="0.6" diameter="1.27"/>
-<via x="50.8" y="3.81" extent="1-16" drill="0.6" diameter="1.27"/>
-<via x="53.34" y="3.81" extent="1-16" drill="0.6" diameter="1.27"/>
 <via x="2.54" y="50.8" extent="1-16" drill="0.6" diameter="1.27"/>
 <via x="6.35" y="55.88" extent="1-16" drill="0.6" diameter="1.27"/>
-<via x="67.31" y="16.51" extent="1-16" drill="0.6" diameter="1.27"/>
 <via x="36.83" y="11.43" extent="1-16" drill="0.6" diameter="1.27"/>
 <contactref element="IC5" pad="P$10"/>
@@
 <via x="37.17925" y="35.052" extent="1-16" drill="0.3" diameter="0.254"/>
 <contactref element="IC2" pad="3"/>
+<via x="35.56" y="3.81" extent="1-16" drill="0.6" diameter="1.27"/>
+<via x="38.1" y="3.81" extent="1-16" drill="0.6" diameter="1.27"/>
+<via x="40.64" y="3.81" extent="1-16" drill="0.6" diameter="1.27"/>
+<via x="43.18" y="3.81" extent="1-16" drill="0.6" diameter="1.27"/>
+<via x="45.72" y="3.81" extent="1-16" drill="0.6" diameter="1.27"/>
+<via x="48.26" y="3.81" extent="1-16" drill="0.6" diameter="1.27"/>
+<via x="50.8" y="3.81" extent="1-16" drill="0.6" diameter="1.27"/>
+<via x="53.34" y="3.81" extent="1-16" drill="0.6" diameter="1.27"/>
 </signal>
 <signal name="+12V" class="1">
@@
 <contactref element="C2" pad="+"/>
 <polygon width="0.3048" layer="1" thermals="no">
-<vertex x="61.31" y="13.843"/>
-<vertex x="79.883" y="13.843"/>
+<vertex x="61.31" y="18.288"/>
+<vertex x="79.883" y="18.288"/>
 <vertex x="79.883" y="0"/>
 <vertex x="61.31" y="0"/>
@@
 <wire x1="36.83" y1="8.89" x2="62.23" y2="8.89" width="1.4224" layer="1"/>
 <wire x1="25.4" y1="69.85" x2="76.2" y2="69.85" width="1.27" layer="1"/>
-<wire x1="78.74" y1="67.31" x2="78.74" y2="34.29" width="1.27" layer="1"/>
 <contactref element="PCB1" pad="VIN"/>
-<wire x1="78.74" y1="34.29" x2="78.74" y2="10.668" width="1.27" layer="1"/>
 <contactref element="C3" pad="1"/>
 <wire x1="23.8368" y1="65.7225" x2="23.83155" y2="68.3768" width="1.27" layer="1"/>
@@
 <wire x1="34.95425" y1="11.14175" x2="34.925" y2="11.1125" width="0.8128" layer="1"/>
 <polygon width="0.254" layer="16" thermals="no">
-<vertex x="61.31" y="13.843"/>
-<vertex x="79.883" y="13.843"/>
+<vertex x="61.31" y="18.288"/>
+<vertex x="79.883" y="18.288"/>
 <vertex x="79.883" y="0"/>
 <vertex x="61.31" y="0"/>
@@
 <via x="78.74" y="11.43" extent="1-16" drill="0.4" diameter="1.27"/>
 <via x="66.04" y="11.43" extent="1-16" drill="0.4" diameter="1.27"/>
-<via x="63.5" y="6.35" extent="1-16" drill="0.4" diameter="1.27"/>
-<via x="63.627" y="8.255" extent="1-16" drill="0.4" diameter="1.27"/>
-<via x="62.611" y="11.43" extent="1-16" drill="0.4" diameter="1.27"/>
-<via x="63.5" y="1.27" extent="1-16" drill="0.4" diameter="1.27"/>
+<via x="62.23" y="17.145" extent="1-16" drill="0.4" diameter="1.27"/>
+<via x="73.66" y="11.43" extent="1-16" drill="0.4" diameter="1.27"/>
+<via x="67.3735" y="17.145" extent="1-16" drill="0.4" diameter="1.27"/>
+<via x="76.2" y="11.43" extent="1-16" drill="0.4" diameter="1.27"/>
 <wire x1="34.9225" y1="13.5255" x2="34.925" y2="13.5255" width="0.8128" layer="1"/>
 <wire x1="34.925" y1="13.5255" x2="34.925" y2="11.1125" width="0.8128" layer="1"/>
 <wire x1="34.925" y1="8.697" x2="34.925" y2="11.1125" width="0.8128" layer="1"/>
+<wire x1="78.74" y1="67.31" x2="78.74" y2="16.8275" width="1.27" layer="1"/>
 </signal>
 <signal name="SHUTTER_OPENED">
@@
 <wire x1="1.93675" y1="43.5" x2="1.93675" y2="41.17725" width="0.6096" layer="1"/>
 <contactref element="IC3" pad="4"/>
-<wire x1="62.23" y1="25.4" x2="62.23" y2="19.05" width="0.4064" layer="1"/>
-<wire x1="62.23" y1="19.05" x2="59.69" y2="16.51" width="0.4064" layer="1"/>
 <wire x1="59.69" y1="16.51" x2="59.69" y2="15.24" width="0.4064" layer="1"/>
 <via x="59.69" y="15.24" extent="1-16" drill="0.3"/>
@@
 <wire x1="24.1173" y1="13.5636" x2="24.65921875" y2="13.5636" width="0.254" layer="1"/>
 <wire x1="24.65921875" y1="13.5636" x2="24.751434375" y2="13.655815625" width="0.254" layer="1"/>
+<wire x1="59.69" y1="16.51" x2="59.69" y2="19.05" width="0.4064" layer="1"/>
+<wire x1="59.69" y1="19.05" x2="62.23" y2="21.59" width="0.4064" layer="1"/>
+<wire x1="62.23" y1="21.59" x2="62.23" y2="24.92125" width="0.4064" layer="1"/>
+<wire x1="62.23" y1="24.92125" x2="61.9735" y2="25.17775" width="0.4064" layer="1"/>
 </signal>
 <signal name="RG-11-IN_5V">
