File: Hardware/RTI-Dome-eth-ENC.brd (EAGLE design)
At the start: 119.4 x 71.1 mm, 77 parts, among them IC1 24AA128ST, IC3 FT232RL, IC4 REG1117, IC5 74LVC245, IC6 74ABT245, J1 POWERPOLE_POWER45A, X13 PN61729-S, X2 J1011F21PNL

Commit message: Change oscilator package reference.
Parts:
- 25MHZ: device rti:CB3 -> rti:SMD-7050_4P
Changed lines of the file:
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@@
 <element name="C17" library="rti" package="C0805" value="100nF" x="75.285" y="22.365" rot="R270"/>
 <element name="J1" library="powerpoles" package="POWERPOLE_PAIR_45A" value="POWERPOLE_POWER45A" x="102.87" y="8.89" rot="MR90"/>
-<element name="25MHZ" library="rti" package="CB3" value="CB3LV-OSCILATOR" x="63.945" y="21.105">
+<element name="25MHZ" library="rti" package="SMD-7050_4P" value="CB3LV-OSCILATOR" x="63.945" y="21.105">
 <attribute name="MPN" value="O705025MEDH4MI" x="63.945" y="21.105" size="1.778" layer="27" display="off"/>
 </element>
