File: Hardware/RTI-Dome-eth-ENC.brd (EAGLE design)
At the start: 119.4 x 71.2 mm, 86 parts, among them IC1 24AA128ST, IC3 FT232RL, IC4 REG1117, IC5 74LVC245, IC6 74ABT245, J1 POWERPOLE_POWER45A, U1 W5500, X13 PN61729-S, X9 J1011F21PNL

Commit message: Revert "Cleanup unused boards and sketches"
This reverts commit 55a3d73229767f07f24b7c99b357f5ead4999c3a.
Parts:
- removed C15: 6.8nF, rti:C0805
- removed C19: 4.7uF, rti:C0805
- removed R25, R26, R27: 49.9 1%, rti:R0805
- removed R28, R29: 330, rti:R0805
- removed R30, R32, R40: 4.7K, rti:R0805
- removed U1: W5500, W5500:LQFP48
- added R22: 4.7K, rti:R0805
- added U$5: ENC424J600-I/PT, Microchip_By_element14_Batch_1:QFP50P1200X1200X120-44N
- 25MHZ: device rti:CB3 -> rti:SMD-7050_4P
- C10: value 22nF -> 10uF
- C12: value 100nF -> 10nF
- C18: value 10nF -> 6.8nF
- C25, C26: device rti:C0805 -> rti:C1206
- R23: value 10 1% -> 10K
- R24: value 49.9 1% -> 12.4K 1%
- R31: value 4.7K -> 10K
- R33: value 4.7K -> 10 1%
- R34, R35, R36, R37: value 4.7K -> 49.9 1%
- R38: value 4.7K -> 1K
- R39: value 12.4K 1% -> 1K
- moved C25 55.1 mm to (89.5, 58.0), turned to 90 degrees
- moved IC4 50.4 mm to (91.7, 51.0)
- moved C26 50.2 mm to (92.0, 58.0)
- moved U$4 48.4 mm to (38.9, 2.71)
- moved C18 34.5 mm to (96.7, 27.7), turned to 0 degrees
- moved FL1 33.8 mm to (95.5, 43.4), turned to 0 degrees
- moved C10 31.4 mm to (68.0, 43.2), turned to 270 degrees
- moved R34 29.1 mm to (91.7, 38.7), turned to 180 degrees
- moved R33 28.9 mm to (91.7, 34.3), turned to 180 degrees
- moved R35 26.2 mm to (91.7, 36.5), turned to 180 degrees
- moved R24 24.4 mm to (70.9, 22.4), turned to 90 degrees
- moved R31 23.3 mm to (72.5, 43.2), turned to 90 degrees
- moved C12 22.5 mm to (91.7, 32.1), turned to 180 degrees
- moved R23 21.1 mm to (79.1, 44.1)
- moved R36 20.4 mm to (91.7, 25.5), turned to 180 degrees
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- renumbered X9 to X2
Connections:
- removed net ACT_LED: U1.27, X2.11
- removed net N$11: C15.2, X2.7
- removed net N$17 (its old number): U1.26
- removed net N$22: R31.1, U1.38
- removed net N$23: R32.1, U1.39
- removed net N$24: R33.1, U1.40
- removed net N$25: R34.1, U1.41
- removed net N$26: R35.1, U1.42
- removed net N$27: R36.1, U1.43
- removed net N$28: R37.1, U1.44
- removed net N$29: R38.1, U1.45
- removed net N$31: C19.2, U1.20
- removed net N$32: U1.18
- removed net N$33: C18.2, U1.22
- removed net N$34: R39.1, U1.10
- removed net N$35: R40.2, U1.23
- removed net XO: U1.31
- new net ACTIVITY: R38.2, U$5.9
- new net BUF_EN: IC5.P$19, R22.2, U$1.A3
- new net N$14: R38.1, X2.12
- new net N$16: C18.2, X2.7
- new net N$18: C12.1, R33.1, X2.3
- net +12V: no longer C25.1, IC4.3
- net +3V3: now also C11.1, C14.1, C17.1, R23.2, R31.2, U$5.12, U$5.15, U$5.18, U$5.4, U$5.44; no longer R28.2, R29.2, R30.2, R36.2, R37.2, R38.2, U1.28
- net 3.3V: now also R22.1
- net AVDD: now also R33.2, R34.2, R35.2; no longer C11.1, C12.1, C14.1, C17.1, R23.2, R24.2, R25.2, U1.11, U1.15, U1.17, U1.21, U1.4, U1.8
- net ETH_CS: now also R31.1, U$5.34; no longer U1.32
- net ETH_RESET: no longer R30.1, U1.37
- net GND: now also C10.1, R24.1, U$5.1, U$5.13, U$5.14, U$5.19, U$5.22, U$5.33, U$5.42, X2.10, X2.11; no longer C10.2, C18.1, C19.1, IC5.P$19, R31.2, R32.2, R33.2, R34.2, R35.2, R39.2, R40.1, U1.14, U1.16, U1.19, U1.29, U1.3, U1.48, U1.9
- net INT_N: now also R23.1, U$5.24; no longer U1.36
- net LINK_ACK: now also R39.2, U$5.10; no longer U1.25, X2.10
- net N$10: now also R39.1, X2.9; no longer R28.1, X2.12
- net N$13: now also C22.1, R36.2, R37.2, X2.6; no longer C10.1, R23.1, X2.3
- net N$7: now also R24.2, U$5.11; no longer C22.1, R26.2, R27.2, X2.6
- net N$8: now also C10.2, U$5.43; no longer R29.1, X2.9
- net RXN: now also R36.1, U$5.21; no longer R26.1, U1.5
- net RXP: now also C18.1, R37.1, U$5.20; no longer C15.1, R27.1, U1.6
- net SCLK: now also U$5.37; no longer U1.33
- net SDI: now also U$5.35; no longer U1.34
- net SDO: now also U$5.36; no longer U1.35
- net TXN: now also R35.1, U$5.17; no longer R25.1, U1.1
- net TXP: now also R34.1, U$5.16; no longer R24.1, U1.2
- net VCC: now also C25.1, IC4.3
- net XI: now also U$5.3; no longer U1.30
Routing:
- net AVDD: track 96.8 -> 20.6 mm
- net BUF_EN: track 0.00 -> 54.2 mm, vias 0 -> 2
- net ACT_LED: track 48.9 -> 0.00 mm, vias 1 -> 0
- net ETH_RESET: track 46.6 -> 0.00 mm, vias 1 -> 0
- net N$7: track 30.8 -> 4.28 mm, vias 3 -> 0
- net +12V: track 239.2 -> 213.5 mm, vias 34 -> 33
- net INT_N: track 43.4 -> 18.7 mm, vias 0 -> 2
- net +3V3: track 146.7 -> 170.7 mm
- net ACTIVITY: track 0.00 -> 23.8 mm, vias 0 -> 2
- net LINK_ACK: track 45.7 -> 30.0 mm, vias 1 -> 2
- net N$18: track 0.00 -> 15.5 mm
- net ETH_CS: track 25.5 -> 39.7 mm, vias 1 -> 2
- net N$13: track 10.0 -> 24.2 mm, vias 0 -> 2
- net VCC: track 134.2 -> 145.8 mm
- net TX2: track 54.2 -> 65.5 mm, vias 0 -> 2
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Other:
- board size 119.4 x 71.2 mm -> 119.4 x 71.1 mm
- board text added: "East / Open"
- board text added: "Home/Closed"
- board text added: "West / Close"
- board text removed: "+5V"
- board text removed: "DIR"
- board text removed: "EN"
- board text removed: "East"
- board text removed: "Home"
- board text removed: "STEP"
- board text removed: "West"
