File: Hardware/RTI-Dome.sch (EAGLE design)
At the start: 50 parts, among them IC1 24AA128ST, IC2 MCP120T-270I_TT, IC3 FT232RL, IC5 74LVC245, IC6 74ABT245, X13 PN61729-S

Commit message: PCB optimisation
Parts:
- removed X12: (no value), con-ptr500:AK500/2
Connections:
- net GND: no longer X12-1.KL, X12-2.KL
Changed lines of the file:
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@@
 <part name="R3" library="rti" deviceset="R-EU" device="'0805'" value="1K"/>
 <part name="C5" library="rti" deviceset="C-EU" device="'0805'" value="100nF"/>
-<part name="X12" library="con-ptr500" deviceset="AK500/2" device=""/>
 <part name="IC3" library="ftdichip" deviceset="FT232R" device="L"/>
 <part name="GND10" library="supply1" deviceset="GND" device=""/>
@@
 <instance part="R3" gate="G$1" x="40.64" y="248.92" rot="R90"/>
 <instance part="C5" gate="G$1" x="114.3" y="180.34"/>
-<instance part="X12" gate="-1" x="378.46" y="129.54" rot="R180"/>
-<instance part="X12" gate="-2" x="378.46" y="134.62" rot="R180"/>
 <instance part="IC3" gate="1" x="289.56" y="149.86"/>
 <instance part="GND10" gate="1" x="274.32" y="111.76"/>
@@
 </segment>
 <segment>
-<pinref part="X12" gate="-1" pin="KL"/>
-<wire x1="370.84" y1="129.54" x2="373.38" y2="129.54" width="0.1524" layer="91"/>
-<label x="370.84" y="129.54" size="1.016" layer="95" rot="R180" xref="yes"/>
-</segment>
-<segment>
 <wire x1="116.84" y1="243.84" x2="119.38" y2="243.84" width="0.1524" layer="91"/>
 <label x="116.84" y="243.84" size="0.8128" layer="95" rot="R180" xref="yes"/>
@@
 </segment>
 <segment>
-<pinref part="X12" gate="-2" pin="KL"/>
-<wire x1="370.84" y1="134.62" x2="373.38" y2="134.62" width="0.1524" layer="91"/>
-<label x="370.84" y="134.62" size="1.016" layer="95" rot="R180" xref="yes"/>
-</segment>
-<segment>

Commit message: Fix some componenent manufacturer reference
Parts:
- IC6: device rti:74LVC245 -> rti:74ABT245
Changed lines of the file:
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@@
 <part name="X6" library="con-ptr500" deviceset="AK500/6" device=""/>
 <part name="IC5" library="rti" deviceset="74*245" device="" technology="LVC"/>
-<part name="IC6" library="rti" deviceset="74*245" device="" technology="LVC" value="74ABT245"/>
+<part name="IC6" library="rti" deviceset="74*245" device="" technology="ABT" value="74ABT245"/>
 <part name="GND7" library="supply1" deviceset="GND" device=""/>
 <part name="R22" library="rti" deviceset="R-EU" device="'0805'" value="4.7K"/>
