File: Hardware/RTI-Dome-eth-ENC.sch (EAGLE design)
At the start: 50 parts, among them IC1 24AA128ST, IC2 MCP120T-270I_TT, IC3 FT232RL, IC5 74LVC245, IC6 74ABT245, X13 PN61729-S

Commit message: Better homing code. Does necessarily stop at home bug sinf home via an interrupt. I'll add more got to go back home after passing it. It does however return the proper position after homing. Added more board for ENC424J600 ethernet chip. Fix position of the headers.
Parts:
- removed IC2: MCP120T-270I_TT, MCP120T-270I_TT:MCP120T-270I_TT
- removed PCB1: ARDUINO_DUE_SHIELD_SHORT, arduino_shield:ARDUINO_DUE_SHIELD_SHORT
- removed X12: (no value), con-ptr500:AK500/2
- added 25MHZ: CB3LV-OSCILATOR, rti:CB3LV-OSCILATOR
- added C10: 10uF, rti:C-EU'0805'
- added C11, C14, C16, C17, C20: 100nF, rti:C-EU'0805'
- added C12, C13, C22: 10nF, rti:C-EU'0805'
- added C18, C21: 6.8nF, rti:C-EU'0805'
- added C25, C26: 10uF, rti:C-EU'1206'
- added FL1: BLM21AG121SN1D, BLM21AG121SN1D:BLM21AG121SN1D
- added IC4: REG1117, burr-brown:REG1117
- added J1: POWERPOLE_POWER45A, powerpoles:POWERPOLE_POWER45A
- added R23, R31: 10K, rti:R-EU'0805'
- added R24: 12.4K 1%, rti:R-EU'0805'
- added R33: 10 1%, rti:R-EU'0805'
- added R34, R35, R36, R37: 49.9 1%, rti:R-EU'0805'
- added R38, R39: 1K, rti:R-EU'0805'
- added U$1: ARDUINO_DUE_SHIELD_FULL, arduino_shield:ARDUINO_DUE_SHIELD_FULL
- added U$2: MCP120T-270I_TT, MCP120T-270I_TT:MCP120T-270I_TT
- added U$5: ENC424J600-I/PT, Microchip_By_element14_Batch_1:ENC424J600-I/PT
- X2: value (none) -> J1011F21PNL; device con-ptr500:AK500/2 -> rti:J1011F21PNL
Connections:
- new net +3V3: 25MHZ.OE, 25MHZ.VDD, C11.1, C13.1, C14.1, C16.1, C17.1, C20.1, C26.1, C9.1, FL1.2, IC3.VCCIO, IC4.VOUT, R23.2, R31.2, U$5.VDD, U$5.VDDOSC, U$5.VDDPLL, U$5.VDDRX, U$5.VDDTX
- new net ACTIVITY: R38.2, U$5.LEDB
- new net AVDD: FL1.1, R33.2, R34.2, R35.2
- new net ETH_CS: R31.1, U$1.52, U$5.~CS/CS
- new net ETH_RESET: U$1.53
- new net INT_N: R23.1, U$1.32, U$5.~INT/SPISEL
- new net LINK_ACK: R39.2, U$5.LEDA
- new net N$10: R39.1, X2.A-R
- new net N$13: C22.1, R36.2, R37.2, X2.CR
- new net N$14: R38.1, X2.AL
- new net N$16: C18.2, X2.RD+
- new net N$17: C21.2, X2.RD-
- new net N$18: C12.1, R33.1, X2.CT
- new net N$7: R24.2, U$5.RBIAS
- new net N$8: C10.2, U$5.VCAP
- new net RXN: C21.1, R36.1, U$5.TPOUT-
- new net RXP: C18.1, R37.1, U$5.TPOUT+
- new net SCLK: U$1.SCK, U$5.SCK/AL
- new net SDI: U$1.SDI, U$5.SO/WR/EN
- new net SDO: U$1.SDO, U$5.SI/RD/R~W
- new net TXN: R35.1, U$5.TPIN-, X2.TD-
- new net TXP: R34.1, U$5.TPIN+, X2.TD+
- new net XI: 25MHZ.FO, U$5.OSC1
- net +12V: now also J1.V+, U$1.VIN; no longer PCB1.VIN, X2-1.KL
- net 3.3V: now also U$1.3.3V, U$2.VDD; no longer C9.1, IC2.VDD, IC3.VCCIO, PCB1.3.3V
- net AT_PARK_PIN: now also U$1.A5; no longer PCB1.A5
- net AT_PARK_PIN_LOOP: now also U$1.A4; no longer PCB1.A4
- net BUF_EN: now also U$1.A3; no longer PCB1.A3
- net BUTTON_EAST_OPEN: now also U$1.5; no longer PCB1.5
- net BUTTON_WEST_CLOSE: now also U$1.6; no longer PCB1.6
- net D13: now also U$1.13; no longer PCB1.13
- net GND: now also 25MHZ.GND, C10.1, C11.2, C12.2, C13.2, C14.2, C16.2, C17.2, C20.2, C22.2, C25.2, C26.2, IC4.GND, J1.GND, R24.1, U$1.GND, U$1.GND@2, U$1.GND@3, U$1.GND@4, U$1.GND@5, U$1.GND@6, U$2.VSS, U$5.VSS, U$5.VSSOSC, U$5.VSSPLL, U$5.VSSRX, U$5.VSSTX, U$5.VSSTX_2, U$5.VSS_2, X2.4/NC, X2.5/NC, X2.C-L, X2.C-R, X2.CGND, X2.CGND2; no longer IC2.VSS, PCB1.GND, PCB1.GND., PCB1.GND.., X12-1.KL, X12-2.KL, X2-2.KL
- net HOME_SHUTTER_CLOSED: now also U$1.2; no longer PCB1.2
- net M_DIR: now also U$1.11; no longer PCB1.11
- net M_EN: now also U$1.10; no longer PCB1.10
- net M_STEP: now also U$1.12; no longer PCB1.12
- net RESET: now also U$1.RESET, U$2.~RST; no longer IC2.~RST, PCB1.RESET
- net RG-11: now also U$1.7; no longer PCB1.7
- net RX2: now also U$1.17(RX2); no longer PCB1.17(RX2)
- net SCL: now also U$1.SCL1; no longer PCB1.SCL1
- net SDA: now also U$1.SDA1; no longer PCB1.SDA1
- net SHUTTER_OPENED: now also U$1.3; no longer PCB1.3
- net TX2: now also U$1.16(TX2); no longer PCB1.16(TX2)
- net VCC: now also C25.1, IC4.VIN, U$1.+5V@3, U$1.+5V@4, U$1.5V; no longer PCB1.5V
- net VPIN: now also U$1.A0; no longer PCB1.A0
- net XBEE_DIN: now also U$1.18(TX1); no longer PCB1.18(TX1)
- net XBEE_DOUT: now also U$1.19(RX1); no longer PCB1.19(RX1)
- net XBEE_RESET: now also U$1.8; no longer PCB1.8

Commit message: Fix some componenent manufacturer reference
Parts:
- 25MHZ: MPN (none) -> O705025MEDH4MI
- IC4: MPN (none) -> REG1117-3.3/2K5
- IC5: MPN (none) -> 74LVC245APW,118
- IC6: device rti:74LVC245 -> rti:74ABT245; MPN (none) -> SN74ABT245BDWR
- U$2: MPN (none) -> MCP120T-270I/TT
- U$5: MPN (none) -> ENC424J600-I/PT
Changed lines of the file:
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@@
 <part name="FRAME1" library="frames" deviceset="DINA3_L" device=""/>
 <part name="X6" library="con-ptr500" deviceset="AK500/6" device=""/>
-<part name="IC5" library="rti" deviceset="74*245" device="" technology="LVC"/>
-<part name="IC6" library="rti" deviceset="74*245" device="" technology="LVC" value="74ABT245"/>
+<part name="IC5" library="rti" deviceset="74*245" device="" technology="LVC">
+<attribute name="MPN" value="74LVC245APW,118"/>
+</part>
+<part name="IC6" library="rti" deviceset="74*245" device="" technology="ABT" value="74ABT245">
+<attribute name="MPN" value="SN74ABT245BDWR"/>
+</part>
 <part name="GND7" library="supply1" deviceset="GND" device=""/>
 <part name="R22" library="rti" deviceset="R-EU" device="'0805'" value="4.7K"/>
@@
 <part name="J1" library="powerpoles" deviceset="POWERPOLE_POWER" device="45A"/>
 <part name="GND15" library="supply1" deviceset="GND" device=""/>
-<part name="25MHZ" library="rti" deviceset="CB3LV-OSCILATOR" device=""/>
+<part name="25MHZ" library="rti" deviceset="CB3LV-OSCILATOR" device="">
+<attribute name="MPN" value="O705025MEDH4MI"/>
+</part>
 <part name="C20" library="rti" deviceset="C-EU" device="'0805'" value="100nF"/>
 <part name="GND17" library="supply1" deviceset="GND" device=""/>
-<part name="U$2" library="MCP120T-270I_TT" deviceset="MCP120T-270I_TT" device=""/>
+<part name="U$2" library="MCP120T-270I_TT" deviceset="MCP120T-270I_TT" device="">
+<attribute name="MPN" value="MCP120T-270I/TT"/>
+</part>
 <part name="GND18" library="supply1" deviceset="GND" device=""/>
 <part name="C13" library="rti" deviceset="C-EU" device="'0805'" value="10nF"/>
@@
 <part name="C11" library="rti" deviceset="C-EU" device="'0805'" value="100nF"/>
 <part name="R31" library="rti" deviceset="R-EU" device="'0805'" value="10K"/>
-<part name="IC4" library="burr-brown" deviceset="REG1117" device=""/>
+<part name="IC4" library="burr-brown" deviceset="REG1117" device="">
+<attribute name="MPN" value="REG1117-3.3/2K5"/>
+</part>
 <part name="+3V1" library="supply1" deviceset="+3V3" device=""/>
 <part name="P+13" library="supply1" deviceset="VCC" device=""/>
@@
 <part name="GND23" library="supply1" deviceset="GND" device=""/>
 <part name="GND13" library="supply1" deviceset="GND" device=""/>
-<part name="U$5" library="Microchip_By_element14_Batch_1" deviceset="ENC424J600-I/PT" device=""/>
+<part name="U$5" library="Microchip_By_element14_Batch_1" deviceset="ENC424J600-I/PT" device="">
+<attribute name="MPN" value="ENC424J600-I/PT"/>
+</part>
 <part name="GND16" library="supply1" deviceset="GND" device=""/>
 <part name="R23" library="rti" deviceset="R-EU" device="'0805'" value="10K"/>
@@
 <instance part="X6" gate="-5" x="345.44" y="185.42" rot="R180"/>
 <instance part="X6" gate="-6" x="345.44" y="190.5" rot="R180"/>
-<instance part="IC5" gate="G$1" x="132.08" y="241.3"/>
-<instance part="IC6" gate="G$1" x="203.2" y="243.84"/>
+<instance part="IC5" gate="G$1" x="132.08" y="241.3">
+<attribute name="MPN" x="132.08" y="241.3" size="1.778" layer="96" display="off"/>
+</instance>
+<instance part="IC6" gate="G$1" x="203.2" y="243.84">
+<attribute name="MPN" x="203.2" y="243.84" size="1.778" layer="96" display="off"/>
+</instance>
 <instance part="IC5" gate="P" x="132.08" y="180.34" rot="R270"/>
 <instance part="IC6" gate="P" x="203.2" y="180.34" rot="R270"/>
@@
 <instance part="GND9" gate="1" x="109.22" y="10.16"/>
 <instance part="J1" gate="G$1" x="378.46" y="83.82"/>
-<instance part="U$2" gate="G$1" x="53.34" y="63.5"/>
+<instance part="U$2" gate="G$1" x="53.34" y="63.5">
+<attribute name="MPN" x="53.34" y="63.5" size="1.778" layer="96" display="off"/>
+</instance>
 <instance part="GND18" gate="1" x="38.1" y="55.88"/>
 </instances>
@@
 <instance part="GND14" gate="1" x="127" y="10.16"/>
 <instance part="GND15" gate="1" x="218.44" y="81.28"/>
-<instance part="25MHZ" gate="G$1" x="203.2" y="81.28" rot="R180"/>
+<instance part="25MHZ" gate="G$1" x="203.2" y="81.28" rot="R180">
+<attribute name="MPN" x="203.2" y="81.28" size="1.778" layer="96" rot="R180" display="off"/>
+</instance>
 <instance part="C20" gate="G$1" x="223.52" y="63.5"/>
 <instance part="GND17" gate="1" x="223.52" y="53.34"/>
