File: Hardware/RTI-Dome-eth-ENC.sch (EAGLE design)
At the start: 86 parts, among them IC1 24AA128ST, IC3 FT232RL, IC4 REG1117, IC5 74LVC245, IC6 74ABT245, J1 POWERPOLE_POWER45A, U1 W5500, X13 PN61729-S, X9 J1011F21PNL

Commit message: Revert "Cleanup unused boards and sketches"
This reverts commit 55a3d73229767f07f24b7c99b357f5ead4999c3a.
Parts:
- removed C15: 6.8nF, rti:C-EU'0805'
- removed C19: 4.7uF, rti:C-EU'0805'
- removed R25, R26, R27: 49.9 1%, rti:R-EU'0805'
- removed R28, R29: 330, rti:R-EU'0805'
- removed R30, R32, R40: 4.7K, rti:R-EU'0805'
- removed U1: W5500, W5500:W5500
- removed X9: J1011F21PNL, rti:J1011F21PNL
- added R22: 4.7K, rti:R-EU'0805'
- added U$5: ENC424J600-I/PT, Microchip_By_element14_Batch_1:ENC424J600-I/PT
- added X2: J1011F21PNL, rti:J1011F21PNL
- 25MHZ: MPN CB3LV-3I-25M0000 -> O705025MEDH4MI
- C1, C3: MPN CC0805KKX5R8BB106 -> (none)
- C10: value 22nF -> 10uF; MPN CC0805JRX7R8BB223 -> (none)
- C11, C14, C16, C17, C20, C4, C5, C6, C7, C8, C9: MPN 0805YD104KAT2A -> (none)
- C12: value 100nF -> 10nF; MPN 0805YD104KAT2A -> (none)
- C13, C22: MPN CC0805KRX7R9BB103 -> (none)
- C18: value 10nF -> 6.8nF; MPN CC0805KRX7R9BB103 -> (none)
- C2: MPN MAL215099804E3 -> (none)
- C21: MPN C0805C682F4HACTU -> (none)
- C25, C26: device rti:C-EU'0805' -> rti:C-EU'1206'; MPN CC0805KKX5R8BB106 -> (none)
- FL1: MPN BLM21AG121SN1D -> (none)
- IC3: MPN FT232RL-REEL -> (none)
- IC5: MPN 74LVC245APW,112 -> 74LVC245APW,118
- IC6: MPN 74ABT245PW,112 -> SN74ABT245BDWR
- R1, R3: MPN RT0805FRE071KL -> (none)
- R10, R2, R6, R7, R8: MPN AT0805BRD07100KL -> (none)
- R11: MPN RT0805FRE0710KL -> (none)
- R12, R13, R14, R15, R16, R17, R18, R19, R20, R21, R4, R9: MPN RT0805FRE074K7L -> (none)
- R23: value 10 1% -> 10K; MPN RT0805FRE1310RL -> (none)
- R24: value 49.9 1% -> 12.4K 1%; MPN RC0805FR-0749R9L -> (none)
- R31: value 4.7K -> 10K; MPN RT0805FRE074K7L -> (none)
- R33: value 4.7K -> 10 1%; MPN RT0805FRE074K7L -> (none)
- R34, R35, R36, R37: value 4.7K -> 49.9 1%; MPN RT0805FRE074K7L -> (none)
- R38: value 4.7K -> 1K; MPN RT0805FRE074K7L -> (none)
- R39: value 12.4K 1% -> 1K; MPN RC0805FR-0712K4L -> (none)
- R5: MPN RT0805FRD07100RL -> (none)
- X1, X11, X3, X8: MPN 691101710002 -> (none)
- X13: MPN SS-52300-001 -> (none)
- X4, X5, X7: MPN 691101710003 -> (none)
- X6: MPN 30.706 -> (none)
Connections:
- removed net ACT_LED: U1.ACTLED, X9.C-L
- removed net N$11: C15.2, X9.RD+
- removed net N$12: C21.2, X9.RD-
- removed net N$22: R31.1, U1.RSVD@2
- removed net N$23: R32.1, U1.RSVD@3
- removed net N$24: R33.1, U1.RSVD@4
- removed net N$25: R34.1, U1.RSVD@5
- removed net N$26: R35.1, U1.RSVD@6
- removed net N$27: R36.1, U1.PMODE2
- removed net N$28: R37.1, U1.PMODE1
- removed net N$29: R38.1, U1.PMODE0
- removed net N$31: C19.2, U1.TOCAP
- removed net N$32: U1.VBG
- removed net N$33: C18.2, U1.1V2O
- removed net N$34: R39.1, U1.EXRES1
- removed net N$35: R40.2, U1.RSVD@1
- removed net XO: U1.XO
- new net ACTIVITY: R38.2, U$5.LEDB
- new net BUF_EN: IC5G$1.*OE, R22.2, U$1.A3
- new net N$14: R38.1, X2.AL
- new net N$16: C18.2, X2.RD+
- new net N$18: C12.1, R33.1, X2.CT
- net +12V: no longer C25.1, IC4.VIN
- net +3V3: now also C11.1, C14.1, C17.1, R23.2, R31.2, U$5.VDD, U$5.VDDOSC, U$5.VDDPLL, U$5.VDDRX, U$5.VDDTX; no longer R28.2, R29.2, R30.2, R36.2, R37.2, R38.2, U1.VDD
- net 3.3V: now also R22.1
- net AVDD: now also R33.2, R34.2, R35.2; no longer C11.1, C12.1, C14.1, C17.1, R23.2, R24.2, R25.2, U1.AVDD@1, U1.AVDD@2, U1.AVDD@3, U1.AVDD@4, U1.AVDD@5, U1.AVDD@6
- net ETH_CS: now also R31.1, U$5.~CS/CS; no longer U1.SCS_N
- net ETH_RESET: no longer R30.1, U1.RST_N
- net GND: now also C10.1, R24.1, U$5.VSS, U$5.VSSOSC, U$5.VSSPLL, U$5.VSSRX, U$5.VSSTX, U$5.VSSTX_2, U$5.VSS_2, X2.4/NC, X2.5/NC, X2.C-L, X2.C-R, X2.CGND, X2.CGND2; no longer C10.2, C18.1, C19.1, IC5G$1.*OE, R31.2, R32.2, R33.2, R34.2, R35.2, R39.2, R40.1, U1.AGND@1, U1.AGND@2, U1.AGND@3, U1.AGND@4, U1.AGND@5, U1.AGND@6, U1.GND, X9.4/NC, X9.5/NC, X9.CGND, X9.CGND2
- net INT_N: now also R23.1, U$5.~INT/SPISEL; no longer U1.INT_N
- net LINK_ACK: now also R39.2, U$5.LEDA; no longer U1.LINKLED, X9.C-R
- net N$10: now also R39.1, X2.A-R; no longer R28.1, X9.AL
- net N$13: now also C22.1, R36.2, R37.2, X2.CR; no longer C10.1, R23.1, X9.CT
- net N$17: now also C21.2, X2.RD-; no longer U1.DUPLED
- net N$7: now also R24.2, U$5.RBIAS; no longer C22.1, R26.2, R27.2, X9.CR
- net N$8: now also C10.2, U$5.VCAP; no longer R29.1, X9.A-R
- net RXN: now also R36.1, U$5.TPOUT-; no longer R26.1, U1.RXN
- net RXP: now also C18.1, R37.1, U$5.TPOUT+; no longer C15.1, R27.1, U1.RXP
- net SCLK: now also U$5.SCK/AL; no longer U1.SCLK
- net SDI: now also U$5.SO/WR/EN; no longer U1.MISO
- net SDO: now also U$5.SI/RD/R~W; no longer U1.MOSI
- net TXN: now also R35.1, U$5.TPIN-, X2.TD-; no longer R25.1, U1.TXN, X9.TD-
- net TXP: now also R34.1, U$5.TPIN+, X2.TD+; no longer R24.1, U1.TXP, X9.TD+
- net VCC: now also C25.1, IC4.VIN
- net XI: now also U$5.OSC1; no longer U1.XI/CLKIN
Other:
- moved on the sheet: 25MHZ, C10, C11, C12, C13, C14, C16, C17, C18, C20, C21, C22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
