File: Hardware/RTI-Dome-eth.brd (EAGLE design)
At the start: 119.4 x 71.2 mm, 85 parts, among them IC1 24AA128ST, IC3 FT232RL, IC4 REG1117, IC5 74LVC245, IC6 74ABT245, J1 POWERPOLE_POWER45A, U1 W5500, X13 PN61729-S, X9 J1011F21PNL

Commit message: Fix a few component values.
Parts:
- 25MHZ: value CB3LV-OSCILATOR -> CB3LV-3I-25M0000
- IC4: value REG1117 -> REG1117-3.3/2K5
- R1, R3: value 1K -> 2.2K
Changed lines of the file:
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@@
 <attribute name="OC_FARNELL" value="unknown" x="-2.9845" y="55.91175" size="1.778" layer="27" display="off"/>
 </element>
-<element name="R1" library="rti" package="R0805" value="1K" x="7.58825" y="44.45" rot="R270">
+<element name="R1" library="rti" package="R0805" value="2.2K" x="7.58825" y="44.45" rot="R270">
 <attribute name="MPN" value="RT0805FRE071KL" x="7.58825" y="44.45" size="1.778" layer="27" rot="R270" display="off"/>
 </element>
-<element name="R3" library="rti" package="R0805" value="1K" x="1.93675" y="44.45" rot="R270">
+<element name="R3" library="rti" package="R0805" value="2.2K" x="1.93675" y="44.45" rot="R270">
 <attribute name="MPN" value="RT0805FRE071KL" x="1.93675" y="44.45" size="1.778" layer="27" rot="R270" display="off"/>
 </element>
@@
 </element>
 <element name="J1" library="powerpoles" package="POWERPOLE_PAIR_45A" value="POWERPOLE_POWER45A" x="102.87" y="8.89" rot="MR90"/>
-<element name="25MHZ" library="rti" package="SMD-7050_4P" value="CB3LV-OSCILATOR" x="58.42" y="27.94">
+<element name="25MHZ" library="rti" package="SMD-7050_4P" value="CB3LV-3I-25M0000" x="58.42" y="27.94">
 <attribute name="MPN" value="CB3LV-3I-25M0000" x="58.42" y="27.94" size="1.778" layer="27" display="off"/>
 </element>
@@
 <attribute name="MPN" value="BLM21AG121SN1D" x="78.74" y="13.97" size="1.778" layer="27" rot="R180" display="off"/>
 </element>
-<element name="IC4" library="burr-brown" package="SOT223" value="REG1117" x="50.8" y="21.59" rot="R180">
+<element name="IC4" library="burr-brown" package="SOT223" value="REG1117-3.3/2K5" x="50.8" y="21.59" rot="R180">
 <attribute name="MPN" value="REG1117-3.3/2K5" x="50.8" y="21.59" size="1.778" layer="27" rot="R180" display="off"/>
 <attribute name="MF" value="" x="50.8" y="21.59" size="1.778" layer="27" rot="R180" display="off"/>
