File: Hardware/RTI-Dome-eth/RTI-Dome-eth.sch (EAGLE design)
At the start: 85 parts, among them IC1 24AA128ST, IC3 FT232RL, IC4 REG1117-3.3/2K5, IC5 74LVC245, IC6 74ABT245, J1 POWERPOLE_POWER45A, U1 W5500, X13 PN61729-S, X9 J1011F21PNL

Commit message: Fix merge conflict
Parts:
- 25MHZ: value CB3LV-3I-25M0000 -> CB3LV-OSCILATOR
- IC4: value REG1117-3.3/2K5 -> REG1117
- R1, R3: value 2.2K -> 1K
Changed lines of the file:
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@@
 <part name="IC1" library="microchip" deviceset="24*" device="ST" technology="AA128"/>
 <part name="GND8" library="supply1" deviceset="GND" device=""/>
-<part name="R1" library="rti" deviceset="R-EU" device="'0805'" value="2.2K">
+<part name="R1" library="rti" deviceset="R-EU" device="'0805'" value="1K">
 <attribute name="MPN" value="RT0805FRE071KL"/>
 </part>
-<part name="R3" library="rti" deviceset="R-EU" device="'0805'" value="2.2K">
+<part name="R3" library="rti" deviceset="R-EU" device="'0805'" value="1K">
 <attribute name="MPN" value="RT0805FRE071KL"/>
 </part>
@@
 <part name="J1" library="powerpoles" deviceset="POWERPOLE_POWER" device="45A"/>
 <part name="GND15" library="supply1" deviceset="GND" device=""/>
-<part name="25MHZ" library="rti" deviceset="CB3LV-OSCILATOR" device="" value="CB3LV-3I-25M0000">
+<part name="25MHZ" library="rti" deviceset="CB3LV-OSCILATOR" device="">
 <attribute name="MPN" value="CB3LV-3I-25M0000"/>
 </part>
@@
 <attribute name="MPN" value="BLM21AG121SN1D"/>
 </part>
-<part name="IC4" library="burr-brown" deviceset="REG1117" device="" value="REG1117-3.3/2K5">
+<part name="IC4" library="burr-brown" deviceset="REG1117" device="">
 <attribute name="MPN" value="REG1117-3.3/2K5"/>
 </part>

Commit message: Fix a  bug when reading number of step per rev after new firnware changes.
Parts:
- removed IC1: 24AA128ST, microchip:24AA128ST
- removed J1: POWERPOLE_POWER45A, powerpoles:POWERPOLE_POWER45A
- removed X6: (no value), con-ptr500:AK500/6
- added IC2: 24LC128T-I_SN, rti:24LC128T-I_SN
- added J2: XT60PW-M, samacsys:XT60PW-M
- added X10, X2: (no value), rti:AK500/3
- C1, C10, C11, C12, C13, C14, C15, C16, C17, C18, C19, C20, C21, C22, C25, C26, C3, C4, C5, C6, C7, C8, C9: device rti:C-EU'0805' -> rcl:C-EUC0805
- C2: device rti:CPOL-EU -> samacsys:MAL215099804E3""
- R1, R10, R11, R12, R13, R14, R15, R16, R17, R18, R19, R2, R20, R21, R23, R24, R25, R26, R27, R28, R29, R3, R30, R31, R32, R33, R34, R35, R36, R37, R38, R39, R4, R40, R5, R6, R7, R8: device rti:R-EU'0805' -> rcl:R-EU_R0805
- U$2: value MCP120T-270I_TT -> MCP120T; device MCP120T-270I_TT:MCP120T-270I_TT -> MCP120T:MCP120T
- X1, X11, X3, X8: device con-ptr500:AK500/2 -> rti:AK500/2
- X13: device con-berg:PN61729-S -> rti:PN61729-S
- X4, X5, X7: device con-ptr500:AK500/3 -> rti:AK500/3
- XB1: device maxstream:XBEE -> rti:XBEE
Connections:
- net +12V: now also J2.2; no longer C25.1, IC4.VIN, J1.V+
- net 3.3V: now also IC2.VCC; no longer IC1.VCC
- net GND: now also IC2.A0, IC2.A1, IC2.A2, IC2.VSS, J2.1; no longer IC1.A0, IC1.A1, IC1.A2, IC1.GND, J1.GND
- net M_DIR_5V: now also X2-3.KL; no longer X6-3.KL
- net M_EN_5V: now also X2-1.KL; no longer X6-1.KL
- net M_STEP_5V: now also X10-2.KL; no longer X6-5.KL
- net SCL: now also IC2.SCL, R1.1; no longer IC1.SCL, R3.1
- net SDA: now also IC2.SDA, R3.1; no longer IC1.SDA, R1.1
- net VCC: now also C25.1, IC4.VIN, X10-1.KL, X10-3.KL, X2-2.KL; no longer X6-2.KL, X6-4.KL, X6-6.KL
Other:
- moved on the sheet: R1, R3
