File: Hardware/RTI-Dome-eth-EPS32/RTI-Dome-eth-ESP32.brd (EAGLE design)
At the start: 111.1 x 76.3 mm, 99 parts, among them IC1 REG1117FA-5.0_500, IC2 24LC64T-I/SN, IC8 REG1117-3.3V, J2 XT60PW-M, T1 MMBT3904LT1, T2 MMBT3904LT1, T3 MMBT3904LT1, U1 W5500, U2 ESP32-DEVKITC-32D, X9 J1011F01PNL

Commit message: ESP32 rotator version routed
Parts:
- added JP1: (no value), rti:JP2
- moved C4 12.3 mm to (32.4, 43.2), turned to 180 degrees
- moved R20 11.9 mm to (43.8, 55.2), turned to 0 degrees
- moved R21 11.4 mm to (43.8, 41.0), turned to 180 degrees
- moved R17 9.47 mm to (43.8, 53.2), turned to 180 degrees
- moved R18 9.05 mm to (43.8, 43.1), turned to 180 degrees
- moved U$3 8.54 mm to (33.7, 48.3), turned to 180 degrees
- moved R4 7.42 mm to (43.8, 51.2), turned to 0 degrees
- moved R15 7.10 mm to (43.8, 45.1), turned to 180 degrees
- moved R9 6.08 mm to (43.8, 49.1), turned to 180 degrees
- moved R16 5.95 mm to (43.8, 47.1), turned to 180 degrees
Connections:
- removed net ETHERNET_CS: U2.29
- removed net N$14: U2.24
- removed net N$40: U2.8
- removed net N$41: U2.9
- removed net N$42: U2.10
- removed net N$43: U2.11
- removed net N$44: U2.12
- removed net N$45: U2.13
- removed net N$46: U2.15
- new net RXD0: JP1.2, U2.34
- new net TXD0: JP1.1, U2.35
- net AT_PARK_PIN: now also U2.24
- net BUTTON_EAST_OPEN: now also U2.11
- net BUTTON_WEST_CLOSE: now also U2.12
- net ETH_CS: now also U2.29
- net GND: now also JP1.3
- net HOME_SHUTTER_CLOSED: now also U2.13
- net RG-11: now also U2.9
- net SHUTTER_OPENED: now also U2.8
- net SPARE1: now also U2.15
- net SPARE2: now also U2.10
Routing:
- net VPIN: track 16.2 -> 84.4 mm, vias 1 -> 0
- net SDO: track 10.8 -> 70.0 mm
- net HOME_SHUTTER_CLOSED_IN_5V: track 2.74 -> 56.5 mm, vias 0 -> 2
- net 3.3V: track 106.3 -> 156.2 mm, vias 3 -> 4
- net ETH_RESET: track 10.2 -> 57.0 mm, vias 1 -> 2
- net SHUTTER_OPENED_IN_5V: track 2.75 -> 48.2 mm, vias 0 -> 2
- net SDI: track 14.6 -> 58.2 mm
- net SCLK: track 8.88 -> 51.3 mm
- net INT_N: track 1.40 -> 43.0 mm, vias 1 -> 2
- net BUTTON_WEST_CLOSE_IN_5V: track 22.7 -> 62.8 mm, vias 1 -> 2
- net ETH_CS: track 11.8 -> 51.4 mm, vias 0 -> 1
- net SPARE1_IN_5V: track 2.74 -> 41.0 mm, vias 0 -> 2
- net RG-11-IN_5V: track 2.74 -> 40.7 mm, vias 0 -> 2
- net AT_PARK_PIN_IN_5V: track 41.7 -> 79.6 mm, vias 1 -> 2
- net BUTTON_EAST_OPEN_5V: track 31.5 -> 69.3 mm, vias 1 -> 2
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Other:
- board text added: "RX"
- board text added: "TX"
