File: Hardware/RTI-Dome-eth-EPS32/RTI-Dome-eth-ESP32.sch (EAGLE design)
At the start: 99 parts, among them IC1 REG1117FA-5.0_500, IC2 24LC64T-I/SN, IC8 REG1117-3.3V, J2 XT60PW-M, T1 MMBT3904LT1, T2 MMBT3904LT1, T3 MMBT3904LT1, U1 W5500, U2 ESP32-DEVKITC-32D, X9 J1011F01PNL

Commit message: ESP32 rotator version routed
Parts:
- added JP1: (no value), rti:JP2E
Connections:
- removed net ETHERNET_CS: U2.IO5
- removed net N$14: U2.IO2
- removed net N$40: U2.IO33
- removed net N$41: U2.IO25
- removed net N$42: U2.IO26
- removed net N$43: U2.IO27
- removed net N$44: U2.IO14
- removed net N$45: U2.IO12
- removed net N$46: U2.IO13
- new net RXD0: JP1.2, U2.RXD0
- new net TXD0: JP1.1, U2.TXD0
- net AT_PARK_PIN: now also U2.IO2
- net BUTTON_EAST_OPEN: now also U2.IO27
- net BUTTON_WEST_CLOSE: now also U2.IO14
- net ETH_CS: now also U2.IO5
- net GND: now also JP1.3
- net HOME_SHUTTER_CLOSED: now also U2.IO12
- net RG-11: now also U2.IO25
- net SHUTTER_OPENED: now also U2.IO33
- net SPARE1: now also U2.IO13
- net SPARE2: now also U2.IO26
Changed lines of the file:
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@@
 <part name="GND3" library="supply1" library_urn="urn:adsk.eagle:library:371" deviceset="GND" device=""/>
 <part name="U2" library="ESP32-DEVKITC-32D" library_urn="urn:adsk.eagle:library:44270575" deviceset="ESP32-DEVKITC-32D" device="" package3d_urn="urn:adsk.eagle:package:44270578/3"/>
+<part name="JP1" library="rti" library_urn="urn:adsk.eagle:library:37256580" deviceset="JP2E" device="" package3d_urn="urn:adsk.eagle:package:37318384/1"/>
+<part name="GND6" library="supply1" library_urn="urn:adsk.eagle:library:371" deviceset="GND" device=""/>
 </parts>
 <sheets>
@@
 <attribute name="NAME" x="96.5028" y="80.6743" size="1.78" layer="95"/>
 <attribute name="VALUE" x="96.5037" y="26.6402" size="1.7799" layer="96"/>
+</instance>
+<instance part="JP1" gate="1" x="168.91" y="71.12" smashed="yes">
+<attribute name="NAME" x="165.1" y="71.12" size="1.778" layer="95" rot="R90"/>
+<attribute name="VALUE" x="174.625" y="71.12" size="1.778" layer="96" rot="R90"/>
+</instance>
+<instance part="GND6" gate="1" x="171.45" y="59.69" smashed="yes">
+<attribute name="VALUE" x="168.91" y="57.15" size="1.778" layer="96"/>
 </instance>
 </instances>
@@
 <label x="134.62" y="77.47" size="1.016" layer="95" xref="yes"/>
 </segment>
+<segment>
+<pinref part="JP1" gate="1" pin="3"/>
+<wire x1="171.45" y1="68.58" x2="171.45" y2="62.23" width="0.1524" layer="91"/>
+<pinref part="GND6" gate="1" pin="GND"/>
+</segment>
 </net>
 <net name="+12V" class="1">
@@
 </segment>
 <segment>
-<wire x1="57.15" y1="15.24" x2="59.69" y2="15.24" width="0.1524" layer="91"/>
-<label x="57.15" y="15.24" size="1.016" layer="95" rot="R180" xref="yes"/>
+<wire x1="88.9" y1="59.69" x2="91.44" y2="59.69" width="0.1524" layer="91"/>
+<label x="88.9" y="59.69" size="1.016" layer="95" rot="R180" xref="yes"/>
+<pinref part="U2" gate="G$1" pin="IO33"/>
 </segment>
 </net>
@@
 </segment>
 <segment>
-<wire x1="57.15" y1="38.1" x2="59.69" y2="38.1" width="0.1524" layer="91"/>
-<label x="57.15" y="38.1" size="1.016" layer="95" rot="R180" xref="yes"/>
+<wire x1="88.9" y1="46.99" x2="91.44" y2="46.99" width="0.1524" layer="91"/>
+<label x="88.9" y="46.99" size="1.016" layer="95" rot="R180" xref="yes"/>
+<pinref part="U2" gate="G$1" pin="IO12"/>
 </segment>
 </net>
@@
 </segment>
 <segment>
-<wire x1="57.15" y1="25.4" x2="59.69" y2="25.4" width="0.1524" layer="91"/>
-<label x="57.15" y="25.4" size="1.016" layer="95" rot="R180" xref="yes"/>
+<wire x1="88.9" y1="52.07" x2="91.44" y2="52.07" width="0.1524" layer="91"/>
+<label x="88.9" y="52.07" size="1.016" layer="95" rot="R180" xref="yes"/>
+<pinref part="U2" gate="G$1" pin="IO27"/>
 </segment>
 </net>
@@
 </segment>
 <segment>
-<wire x1="57.15" y1="27.94" x2="59.69" y2="27.94" width="0.1524" layer="91"/>
-<label x="57.15" y="27.94" size="1.016" layer="95" rot="R180" xref="yes"/>
+<wire x1="88.9" y1="49.53" x2="91.44" y2="49.53" width="0.1524" layer="91"/>
+<label x="88.9" y="49.53" size="1.016" layer="95" rot="R180" xref="yes"/>
+<pinref part="U2" gate="G$1" pin="IO14"/>
 </segment>
 </net>
@@
 </segment>
 <segment>
-<wire x1="57.15" y1="20.32" x2="58.42" y2="20.32" width="0.1524" layer="91"/>
-<wire x1="58.42" y1="20.32" x2="59.69" y2="20.32" width="0.1524" layer="91"/>
-<label x="57.15" y="20.32" size="1.016" layer="95" rot="R180" xref="yes"/>
+<pinref part="U2" gate="G$1" pin="IO25"/>
+<wire x1="88.9" y1="57.15" x2="91.44" y2="57.15" width="0.1524" layer="91"/>
+<label x="88.9" y="57.15" size="1.016" layer="95" ratio="4" rot="R180" xref="yes"/>
 </segment>
 </net>
@@
 </segment>
 <segment>
-<wire x1="57.15" y1="12.7" x2="59.69" y2="12.7" width="0.1524" layer="91"/>
-<label x="57.15" y="12.7" size="1.016" layer="95" rot="R180" xref="yes"/>
+<wire x1="134.62" y1="41.91" x2="132.08" y2="41.91" width="0.1524" layer="91"/>
+<label x="134.62" y="41.91" size="1.016" layer="95" xref="yes"/>
+<pinref part="U2" gate="G$1" pin="IO2"/>
 </segment>
 </net>
@@
 </segment>
 <segment>
-<wire x1="57.15" y1="40.64" x2="59.69" y2="40.64" width="0.1524" layer="91"/>
-<label x="57.15" y="40.64" size="1.016" layer="95" rot="R180" xref="yes"/>
+<wire x1="88.9" y1="41.91" x2="91.44" y2="41.91" width="0.1524" layer="91"/>
+<label x="88.9" y="41.91" size="1.016" layer="95" rot="R180" xref="yes"/>
+<pinref part="U2" gate="G$1" pin="IO13"/>
 </segment>
 </net>
@@
 </segment>
 <segment>
-<wire x1="57.15" y1="22.86" x2="59.69" y2="22.86" width="0.1524" layer="91"/>
-<label x="57.15" y="22.86" size="1.016" layer="95" rot="R180" xref="yes"/>
+<wire x1="88.9" y1="54.61" x2="91.44" y2="54.61" width="0.1524" layer="91"/>
+<label x="88.9" y="54.61" size="1.016" layer="95" rot="R180" xref="yes"/>
+<pinref part="U2" gate="G$1" pin="IO26"/>
 </segment>
 </net>
@@
 </segment>
 </net>
-<net name="ETHERNET_CS" class="0">
+<net name="ETH_CS" class="0">
 <segment>
 <pinref part="U2" gate="G$1" pin="IO5"/>
@@
 </segment>
 </net>
-<net name="N$14" class="0">
-<segment>
-<pinref part="U2" gate="G$1" pin="IO2"/>
-<wire x1="134.62" y1="41.91" x2="132.08" y2="41.91" width="0.1524" layer="91"/>
-</segment>
-</net>
 <net name="N$15" class="0">
 <segment>
@@
 <pinref part="U2" gate="G$1" pin="SENSOR_VN"/>
 <wire x1="88.9" y1="69.85" x2="91.44" y2="69.85" width="0.1524" layer="91"/>
-</segment>
-</net>
-<net name="N$40" class="0">
-<segment>
-<pinref part="U2" gate="G$1" pin="IO33"/>
-<wire x1="88.9" y1="59.69" x2="91.44" y2="59.69" width="0.1524" layer="91"/>
-</segment>
-</net>
-<net name="N$41" class="0">
-<segment>
-<pinref part="U2" gate="G$1" pin="IO25"/>
-<wire x1="88.9" y1="57.15" x2="91.44" y2="57.15" width="0.1524" layer="91"/>
-</segment>
-</net>
-<net name="N$42" class="0">
-<segment>
-<pinref part="U2" gate="G$1" pin="IO26"/>
-<wire x1="88.9" y1="54.61" x2="91.44" y2="54.61" width="0.1524" layer="91"/>
-</segment>
-</net>
-<net name="N$43" class="0">
-<segment>
-<pinref part="U2" gate="G$1" pin="IO27"/>
-<wire x1="88.9" y1="52.07" x2="91.44" y2="52.07" width="0.1524" layer="91"/>
-</segment>
-</net>
-<net name="N$44" class="0">
-<segment>
-<pinref part="U2" gate="G$1" pin="IO14"/>
-<wire x1="88.9" y1="49.53" x2="91.44" y2="49.53" width="0.1524" layer="91"/>
-</segment>
-</net>
-<net name="N$45" class="0">
-<segment>
-<pinref part="U2" gate="G$1" pin="IO12"/>
-<wire x1="88.9" y1="46.99" x2="91.44" y2="46.99" width="0.1524" layer="91"/>
-</segment>
-</net>
-<net name="N$46" class="0">
-<segment>
-<pinref part="U2" gate="G$1" pin="IO13"/>
-<wire x1="88.9" y1="41.91" x2="91.44" y2="41.91" width="0.1524" layer="91"/>
 </segment>
 </net>
@@
 </segment>
 </net>
+<net name="TXD0" class="0">
+<segment>
+<pinref part="U2" gate="G$1" pin="TXD0"/>
+<wire x1="134.62" y1="69.85" x2="132.08" y2="69.85" width="0.1524" layer="91"/>
+<label x="134.62" y="69.85" size="1.016" layer="95" ratio="4" xref="yes"/>
+</segment>
+<segment>
+<pinref part="JP1" gate="1" pin="1"/>
+<wire x1="163.83" y1="66.04" x2="166.37" y2="66.04" width="0.1524" layer="91"/>
+<wire x1="166.37" y1="66.04" x2="166.37" y2="68.58" width="0.1524" layer="91"/>
+<label x="163.83" y="66.04" size="1.016" layer="95" ratio="4" rot="R180" xref="yes"/>
+</segment>
+</net>
+<net name="RXD0" class="0">
+<segment>
+<pinref part="U2" gate="G$1" pin="RXD0"/>
+<wire x1="134.62" y1="67.31" x2="132.08" y2="67.31" width="0.1524" layer="91"/>
+<label x="134.62" y="67.31" size="1.016" layer="95" ratio="4" xref="yes"/>
+</segment>
+<segment>
+<pinref part="JP1" gate="1" pin="2"/>
+<wire x1="163.83" y1="63.5" x2="168.91" y2="63.5" width="0.1524" layer="91"/>
+<wire x1="168.91" y1="63.5" x2="168.91" y2="68.58" width="0.1524" layer="91"/>
+<label x="163.83" y="63.5" size="1.016" layer="95" ratio="4" rot="R180" xref="yes"/>
+</segment>
+</net>
