File: Hardware/RTI-Dome-eth-EPS32/RTI-Dome-eth-ESP32.sch (EAGLE design)
At the start: 100 parts, among them IC1 REG1117FA-5.0_500, IC2 24LC64T-I/SN, IC8 REG1117-3.3V, J2 XT60PW-M, T1 MMBT3904LT1, T2 MMBT3904LT1, T3 MMBT3904LT1, U1 W5500, U2 ESP32-DevKitC ESP32-WROOM-32U, X9 J1011F01PNL

Commit message: Set the proper version of the EXP32 kit for each board.
Parts:
- U2: device ESP32-DEVKITC-32D:ESP32-DEVKITC-32D -> ESP32-DEVKITC-32D:ESP32-DEVKITC-32U
Changed lines of the file:
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@@
 <part name="IC1" library="REG1117FA-5.0_500" library_urn="urn:adsk.eagle:library:43937876" deviceset="REG1117FA-5.0_500" device="" package3d_urn="urn:adsk.eagle:package:43937879/3"/>
 <part name="GND3" library="supply1" library_urn="urn:adsk.eagle:library:371" deviceset="GND" device=""/>
-<part name="U2" library="ESP32-DEVKITC-32D" library_urn="urn:adsk.eagle:library:44270575" deviceset="ESP32-DEVKITC-32D" device="" package3d_urn="urn:adsk.eagle:package:44270578/3" value="ESP32-DevKitC ESP32-WROOM-32U"/>
+<part name="U2" library="ESP32-DEVKITC-32D" library_urn="urn:adsk.eagle:library:44270575" deviceset="ESP32-DEVKITC-32" device="U" package3d_urn="urn:adsk.eagle:package:44294361/2" value="ESP32-DevKitC ESP32-WROOM-32U"/>
 <part name="JP1" library="rti" library_urn="urn:adsk.eagle:library:37256580" deviceset="JP2E" device="" package3d_urn="urn:adsk.eagle:package:37318384/1"/>
 <part name="GND6" library="supply1" library_urn="urn:adsk.eagle:library:371" deviceset="GND" device=""/>

Commit message: Fix pin assignement issues for ESP32
Connections:
- removed net N$15: U2.IO15
- net AT_PARK_PIN: now also U2.IO35; no longer U2.IO2
- net HOME_SHUTTER_CLOSED: now also U2.IO15; no longer U2.IO12
- net M_DIR: now also U2.IO2; no longer U2.IO35
- net M_EN: now also U2.IO13; no longer U2.IO34
- net SPARE1: now also U2.IO34; no longer U2.IO13
Changed lines of the file:
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@@
 </segment>
 <segment>
-<pinref part="U2" gate="G$1" pin="IO34"/>
-<wire x1="88.9" y1="67.31" x2="91.44" y2="67.31" width="0.1524" layer="91"/>
-<label x="88.9" y="67.31" size="1.016" layer="95" rot="R180" xref="yes"/>
+<wire x1="88.9" y1="41.91" x2="91.44" y2="41.91" width="0.1524" layer="91"/>
+<label x="88.9" y="41.91" size="1.016" layer="95" rot="R180" xref="yes"/>
+<pinref part="U2" gate="G$1" pin="IO13"/>
 </segment>
 </net>
@@
 </segment>
 <segment>
-<pinref part="U2" gate="G$1" pin="IO35"/>
-<wire x1="88.9" y1="64.77" x2="91.44" y2="64.77" width="0.1524" layer="91"/>
-<label x="88.9" y="64.77" size="1.016" layer="95" rot="R180" xref="yes"/>
+<wire x1="134.62" y1="41.91" x2="132.08" y2="41.91" width="0.1524" layer="91"/>
+<label x="134.62" y="41.91" size="1.016" layer="95" xref="yes"/>
+<pinref part="U2" gate="G$1" pin="IO2"/>
 </segment>
 </net>
@@
 </segment>
 <segment>
-<wire x1="88.9" y1="46.99" x2="91.44" y2="46.99" width="0.1524" layer="91"/>
-<label x="88.9" y="46.99" size="1.016" layer="95" rot="R180" xref="yes"/>
-<pinref part="U2" gate="G$1" pin="IO12"/>
+<pinref part="U2" gate="G$1" pin="IO15"/>
+<wire x1="134.62" y1="39.37" x2="132.08" y2="39.37" width="0.1524" layer="91"/>
+<label x="134.62" y="39.37" size="1.27" layer="95" xref="yes"/>
 </segment>
 </net>
@@
 </segment>
 <segment>
-<wire x1="134.62" y1="41.91" x2="132.08" y2="41.91" width="0.1524" layer="91"/>
-<label x="134.62" y="41.91" size="1.016" layer="95" xref="yes"/>
-<pinref part="U2" gate="G$1" pin="IO2"/>
+<pinref part="U2" gate="G$1" pin="IO35"/>
+<wire x1="88.9" y1="64.77" x2="91.44" y2="64.77" width="0.1524" layer="91"/>
+<label x="88.9" y="64.77" size="1.016" layer="95" rot="R180" xref="yes"/>
 </segment>
 </net>
@@
 </segment>
 <segment>
-<wire x1="88.9" y1="41.91" x2="91.44" y2="41.91" width="0.1524" layer="91"/>
-<label x="88.9" y="41.91" size="1.016" layer="95" rot="R180" xref="yes"/>
-<pinref part="U2" gate="G$1" pin="IO13"/>
+<pinref part="U2" gate="G$1" pin="IO34"/>
+<wire x1="88.9" y1="67.31" x2="91.44" y2="67.31" width="0.1524" layer="91"/>
+<label x="88.9" y="67.31" size="1.016" layer="95" rot="R180" xref="yes"/>
 </segment>
 </net>
@@
 </segment>
 </net>
-<net name="N$15" class="0">
-<segment>
-<pinref part="U2" gate="G$1" pin="IO15"/>
-<wire x1="134.62" y1="39.37" x2="132.08" y2="39.37" width="0.1524" layer="91"/>
-</segment>
-</net>

Commit message: Fixed a lot of issue with the ESP32 and serial ports.
Alpaca Discovery and API server are now running in their own tasks.
Parts:
- added X7: (no value), rti:AK500/3
Connections:
- new net SPARE_OUT1: U$1G$1.A3, U2.IO0
- new net SPARE_OUT1_5V: U$1G$1.Y3, X7-3.KL
- new net SPARE_OUT2: U$1G$1.A4, U2.IO12
- new net SPARE_OUT2_5V: U$1G$1.Y4, X7-2.KL
- net GND: now also X7-1.KL; no longer U$1G$1.A3, U$1G$1.A4
- net INT_N: no longer U2.IO0
- net RX2: now also JP1.2
- net RXD0: no longer JP1.2
- net TX2: now also JP1.1
- net TXD0: no longer JP1.1
Changed lines of the file:
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@@
 <part name="JP1" library="rti" library_urn="urn:adsk.eagle:library:37256580" deviceset="JP2E" device="" package3d_urn="urn:adsk.eagle:package:37318384/1"/>
 <part name="GND6" library="supply1" library_urn="urn:adsk.eagle:library:371" deviceset="GND" device=""/>
+<part name="X7" library="rti" library_urn="urn:adsk.eagle:library:37256580" deviceset="AK500/3" device="" package3d_urn="urn:adsk.eagle:package:37500967/6"/>
 </parts>
 <sheets>
@@
 <instance part="GND6" gate="1" x="171.45" y="59.69" smashed="yes">
 <attribute name="VALUE" x="168.91" y="57.15" size="1.778" layer="96"/>
+</instance>
+<instance part="X7" gate="-1" x="303.53" y="127" smashed="yes" rot="R180">
+<attribute name="NAME" x="304.8" y="126.111" size="1.778" layer="95"/>
+</instance>
+<instance part="X7" gate="-2" x="303.53" y="132.08" smashed="yes" rot="R180">
+<attribute name="NAME" x="304.8" y="131.191" size="1.778" layer="95"/>
+</instance>
+<instance part="X7" gate="-3" x="303.53" y="137.16" smashed="yes" rot="R180">
+<attribute name="NAME" x="304.8" y="136.271" size="1.778" layer="95"/>
+<attribute name="VALUE" x="307.34" y="140.843" size="1.778" layer="96" rot="R180"/>
 </instance>
 </instances>
@@
 </segment>
 <segment>
-<wire x1="187.96" y1="246.38" x2="190.5" y2="246.38" width="0.1524" layer="91"/>
-<label x="187.96" y="246.38" size="0.8128" layer="95" rot="R180" xref="yes"/>
-<pinref part="U$1" gate="G$1" pin="A4"/>
-</segment>
-<segment>
 <wire x1="187.96" y1="243.84" x2="190.5" y2="243.84" width="0.1524" layer="91"/>
-<label x="187.96" y="243.84" size="0.8128" layer="95" rot="R180" xref="yes"/>
+<label x="187.96" y="243.84" size="1.016" layer="95" rot="R180" xref="yes"/>
 <pinref part="U$1" gate="G$1" pin="A5"/>
 </segment>
 <segment>
 <wire x1="187.96" y1="241.3" x2="190.5" y2="241.3" width="0.1524" layer="91"/>
-<label x="187.96" y="241.3" size="0.8128" layer="95" rot="R180" xref="yes"/>
+<label x="187.96" y="241.3" size="1.016" layer="95" rot="R180" xref="yes"/>
 <pinref part="U$1" gate="G$1" pin="A6"/>
 </segment>
 <segment>
 <wire x1="187.96" y1="238.76" x2="190.5" y2="238.76" width="0.1524" layer="91"/>
-<label x="187.96" y="238.76" size="0.8128" layer="95" rot="R180" xref="yes"/>
+<label x="187.96" y="238.76" size="1.016" layer="95" rot="R180" xref="yes"/>
 <pinref part="U$1" gate="G$1" pin="A7"/>
 </segment>
@@
 </segment>
 <segment>
-<wire x1="187.96" y1="248.92" x2="190.5" y2="248.92" width="0.1524" layer="91"/>
-<label x="187.96" y="248.92" size="1.016" layer="95" rot="R180" xref="yes"/>
-<pinref part="U$1" gate="G$1" pin="A3"/>
-</segment>
-<segment>
 <pinref part="IC1" gate="G$1" pin="GND"/>
 <wire x1="31.75" y1="130.81" x2="31.75" y2="132.08" width="0.1524" layer="91"/>
@@
 <wire x1="171.45" y1="68.58" x2="171.45" y2="62.23" width="0.1524" layer="91"/>
 <pinref part="GND6" gate="1" pin="GND"/>
+</segment>
+<segment>
+<pinref part="X7" gate="-1" pin="KL"/>
+<wire x1="295.91" y1="127" x2="298.45" y2="127" width="0.1524" layer="91"/>
+<label x="295.91" y="127" size="1.016" layer="95" rot="R180" xref="yes"/>
 </segment>
 </net>
@@
 </segment>
 </net>
-<net name="INT_N" class="0">
-<segment>
-<pinref part="U2" gate="G$1" pin="IO0"/>
-<wire x1="134.62" y1="44.45" x2="132.08" y2="44.45" width="0.1524" layer="91"/>
-<label x="134.62" y="44.45" size="1.016" layer="95" xref="yes"/>
-</segment>
-</net>
 <net name="DIR-5V_TR" class="0">
 <segment>
@@
 <label x="134.62" y="52.07" size="1.016" layer="95" xref="yes"/>
 </segment>
-</net>
-<net name="RX2" class="0">
-<segment>
-<pinref part="U2" gate="G$1" pin="IO16"/>
-<wire x1="134.62" y1="49.53" x2="132.08" y2="49.53" width="0.1524" layer="91"/>
-<label x="134.62" y="49.53" size="1.016" layer="95" xref="yes"/>
-</segment>
-</net>
-<net name="TXD0" class="0">
-<segment>
-<pinref part="U2" gate="G$1" pin="TXD0"/>
-<wire x1="134.62" y1="69.85" x2="132.08" y2="69.85" width="0.1524" layer="91"/>
-<label x="134.62" y="69.85" size="1.016" layer="95" ratio="4" xref="yes"/>
-</segment>
 <segment>
 <pinref part="JP1" gate="1" pin="1"/>
@@
 </segment>
 </net>
-<net name="RXD0" class="0">
-<segment>
-<pinref part="U2" gate="G$1" pin="RXD0"/>
-<wire x1="134.62" y1="67.31" x2="132.08" y2="67.31" width="0.1524" layer="91"/>
-<label x="134.62" y="67.31" size="1.016" layer="95" ratio="4" xref="yes"/>
+<net name="RX2" class="0">
+<segment>
+<pinref part="U2" gate="G$1" pin="IO16"/>
+<wire x1="134.62" y1="49.53" x2="132.08" y2="49.53" width="0.1524" layer="91"/>
+<label x="134.62" y="49.53" size="1.016" layer="95" xref="yes"/>
 </segment>
 <segment>
@@
 </segment>
 </net>
+<net name="TXD0" class="0">
+<segment>
+<pinref part="U2" gate="G$1" pin="TXD0"/>
+<wire x1="134.62" y1="69.85" x2="132.08" y2="69.85" width="0.1524" layer="91"/>
+<label x="134.62" y="69.85" size="1.016" layer="95" ratio="4" xref="yes"/>
+</segment>
+</net>
+<net name="RXD0" class="0">
+<segment>
+<pinref part="U2" gate="G$1" pin="RXD0"/>
+<wire x1="134.62" y1="67.31" x2="132.08" y2="67.31" width="0.1524" layer="91"/>
+<label x="134.62" y="67.31" size="1.016" layer="95" ratio="4" xref="yes"/>
+</segment>
+</net>
+<net name="SPARE_OUT1_5V" class="0">
+<segment>
+<pinref part="U$1" gate="G$1" pin="Y3"/>
+<wire x1="218.44" y1="248.92" x2="215.9" y2="248.92" width="0.1524" layer="91"/>
+<label x="218.44" y="248.92" size="1.016" layer="95" xref="yes"/>
+</segment>
+<segment>
+<pinref part="X7" gate="-3" pin="KL"/>
+<wire x1="295.91" y1="137.16" x2="298.45" y2="137.16" width="0.1524" layer="91"/>
+<label x="295.91" y="137.16" size="1.016" layer="95" rot="R180" xref="yes"/>
+</segment>
+</net>
+<net name="SPARE_OUT1" class="0">
+<segment>
+<wire x1="187.96" y1="248.92" x2="190.5" y2="248.92" width="0.1524" layer="91"/>
+<label x="187.96" y="248.92" size="1.016" layer="95" rot="R180" xref="yes"/>
+<pinref part="U$1" gate="G$1" pin="A3"/>
+</segment>
+<segment>
+<pinref part="U2" gate="G$1" pin="IO0"/>
+<wire x1="134.62" y1="44.45" x2="132.08" y2="44.45" width="0.1524" layer="91"/>
+<label x="134.62" y="44.45" size="1.016" layer="95" xref="yes"/>
+</segment>
+</net>
+<net name="SPARE_OUT2" class="0">
+<segment>
+<pinref part="U2" gate="G$1" pin="IO12"/>
+<wire x1="88.9" y1="46.99" x2="91.44" y2="46.99" width="0.1524" layer="91"/>
+<label x="88.9" y="46.99" size="1.016" layer="95" rot="R180" xref="yes"/>
+</segment>
+<segment>
+<wire x1="187.96" y1="246.38" x2="190.5" y2="246.38" width="0.1524" layer="91"/>
+<label x="187.96" y="246.38" size="1.016" layer="95" rot="R180" xref="yes"/>
+<pinref part="U$1" gate="G$1" pin="A4"/>
+</segment>
+</net>
+<net name="SPARE_OUT2_5V" class="0">
+<segment>
+<pinref part="U$1" gate="G$1" pin="Y4"/>
+<wire x1="218.44" y1="246.38" x2="215.9" y2="246.38" width="0.1524" layer="91"/>
+<label x="218.44" y="246.38" size="1.016" layer="95" xref="yes"/>
+</segment>
+<segment>
+<pinref part="X7" gate="-2" pin="KL"/>
+<wire x1="295.91" y1="132.08" x2="298.45" y2="132.08" width="0.1524" layer="91"/>
+<label x="295.91" y="132.08" size="1.016" layer="95" rot="R180" xref="yes"/>
+</segment>
+</net>
