File: Hardware/RTI-Dome-Shutter-ESP32/RTI-Dome-Shutter-ESP32.sch (EAGLE design)
At the start: 65 parts, among them IC1 REG1117FA-5.0_500, IC2 24LC64T-I/SN, IC8 REG1117-3.3V, J1 691313510003, J10 691313510002, J11 691313510002, J12 691313510002, J2 XT60PW-M, J3 691313510003, J4 691313510003, J6 691313510003, J7 691313510003, J8 691313510002, J9 691313510002, U1 ESP32-DEVKITC-32E

Commit message: Adding latest PCB files
Parts:
- removed C2: 100uF, samacsys:MAL215099804E3""
- removed C27, C28, C3, C42: 10uF, rti:C-EU'0603'
- removed C5: 100nF, rti:C-EU'0603'
- removed IC1: REG1117FA-5.0_500, REG1117FA-5.0_500:REG1117FA-5.0_500
- removed IC2: 24LC64T-I/SN, rti:24LC64T-I/SN
- removed J11: 691313510002, samacsys:691313510002
- removed R10, R7, R8: 100K 0.1%, rti:R-EU'0603'
- removed R20: 4.7K, rti:R-EU'0603'
- removed R46: 100, rti:R-EU'0603'
- added C10, C11, C12: 22uF 35V, rcl:C-EUC1206
- added C25: 10uF, rcl:C-EUC0805
- added C26: 22uF, rcl:C-EUC0805
- added C29: 1uF, rcl:C-EUC0805
- added C7: 10uF, rcl:C-EUC1206
- added C8: 0.1uF, rcl:C-EUC1206
- added C9: 3.3nF, rcl:C-EUC0805
- added L1: IHLP1212BZER2R2M11, samacsys:IHLP1212BZER2R2M11
- added PS1: TPS62133RGTR, samacsys:TPS62133RGTR
- added R11: 100K, rcl:R-EU_R0603
- JP1: value (none) -> 3PIN_Header; LCSC_PART (none) -> C19190477
- R1, R3: value 1K -> 100K; MPN RT0805FRE071KL -> RT0805FRD07100RL
- R2: value 100K 0.1% -> 40K 0.1%
- R6: value 100K 0.1% -> 10K 0.1%
- T1, T2, T3: value (none) -> MMBT3904LT1
Connections:
- net BUTTON_EAST_OPEN renamed BUTTON_OPEN
- net BUTTON_EAST_OPEN-IN_EXT renamed BUTTON_OPEN-IN_EXT
- net BUTTON_EAST_OPEN_5V renamed BUTTON_OPEN_5V
- net BUTTON_WEST_CLOSE renamed BUTTON_CLOSE
- net BUTTON_WEST_CLOSE-IN_EXT renamed BUTTON_CLOSE-IN_EXT
- net BUTTON_WEST_CLOSE_IN_5V renamed BUTTON_CLOSE_IN_5V
- net HOME_SHUTTER_CLOSED renamed SHUTTER_CLOSED
- net HOME_SHUTTER_CLOSED-IN_EXT renamed SHUTTER_CLOSED-IN_EXT
- net HOME_SHUTTER_CLOSED_IN_5V renamed SHUTTER_CLOSED_IN_5V
- net SPARE1 renamed LOWER_CLOSED
- net SPARE1-IN_EXT renamed LOWER_CLOSED-IN_EXT
- net SPARE1_IN_5V renamed LOWER_CLOSED_IN_5V
- net SPARE2 renamed LOWER_OPENED
- net SPARE2-IN_EXT renamed LOWER_OPENED-IN_EXT
- net SPARE2_IN_5V renamed LOWER_OPENED_IN_5V
- net SPARE_OUT1_5V renamed LOWER_DIR_5V
- net SPARE_OUT2_5V renamed LOWER_ENABLE_5V
- removed net AT_PARK_PIN: U$3G$1.Y7, U1.IO35
- removed net AT_PARK_PIN-IN_EXT: J11.2, R46.2
- removed net AT_PARK_PIN_IN_5V: C42.1, R20.1, R46.1, U$3G$1.A7
- removed net N$2: R7.2, R8.1
- removed net N$3: R10.1, R8.2
- removed net N$5: R2.2, R7.1
- removed net SPARE_OUT1: U$1G$1.A3, U1.IO0
- removed net SPARE_OUT2: U$1G$1.A4, U1.IO12
- new net LOWER_DIR: R3.2, U$1G$1.A3, U1.IO0
- new net LOWER_ENABLE: R1.2, U$1G$1.A4, U1.IO12
- new net N$1: U$3G$1.Y7
- new net PG: PS1.PG, R11.2
- new net SS/TR: C9.1, PS1.SS/TR
- new net SW: L1.1, PS1.SW_1, PS1.SW_2, PS1.SW_3
- net +12V: now also C10.1, C11.1, C12.1, C7.1, C8.1, PS1.AVIN, PS1.EN, PS1.PVIN_1, PS1.PVIN_2, R2.2; no longer C2.+, C27.1, C3.1, IC1.VIN, R10.2
- net 3.3V: now also R3.1; no longer C5.1, IC2.VCC, R1.2, R3.2
- net GND: now also C10.2, C11.2, C12.2, C25.1, C26.1, C29.1, C7.2, C8.2, C9.2, PS1.AGND, PS1.DEF, PS1.EP, PS1.FB, PS1.FSW, PS1.PGND_1, PS1.PGND_2, R1.1, U$3G$1.A7; no longer C2.-, C27.2, C28.2, C3.2, C42.2, C5.2, IC1.GND, IC2.A0, IC2.A1, IC2.A2, IC2.VSS, J11.1
- net SCL: no longer IC2.SCL, R1.1
- net SDA: no longer IC2.SDA, R3.1
- net VCC: now also C25.2, C26.2, C29.2, L1.2, PS1.VOS, R11.1; no longer C28.1, IC1.VOUT_1, IC1.VOUT_2, R20.2
- net VPIN: now also U1.IO35; no longer U1.SENSOR_VP
Other:
- moved on the sheet: JP1, R1, R2, R3, R6, U1
