File: Hardware/RTI-Dome-eth-ESP32/RTI-Dome-eth-ESP32.brd (EAGLE design)
At the start: 111.1 x 76.3 mm, 102 parts, among them IC2 24LC64T-I/SN, IC8 REG1117-3.3V, J1 691313510003, J10 691313510002, J11 691313510002, J12 691313510002, J2 XT60PW-M, J3 691313510003, J4 691313510003, J6 691313510003, J7 691313510003, J8 691313510002, J9 691313510002, T1 MMBT3904LT1, T2 MMBT3904LT1, T3 MMBT3904LT1, U1 W5500, U2 ESP32-DevKitC-32UE, X9 J1011F01PNL

Commit message: Adding latest PCB files
Parts:
- removed C5: 100nF, rcl:C0603
- removed IC2: 24LC64T-I/SN, rti:SOIC127P600X175-8N
- R1, R3: value 1K -> 100K; device rcl:R0603 -> rti:R0603
- moved R1 36.7 mm to (14.0, 56.5), turned to 0 degrees
- moved R3 22.3 mm to (14.0, 37.0)
- moved C1 1.00 mm to (50.4, 64.8)
- moved C40 1.00 mm to (86.0, 64.8)
- moved C41 1.00 mm to (41.5, 64.8)
- moved C42 1.00 mm to (96.2, 64.8)
- moved C43 1.00 mm to (77.1, 64.8)
- moved C44 1.00 mm to (59.3, 64.8)
- moved C46 1.00 mm to (68.2, 64.8)
- moved R49 1.00 mm to (30.2, 64.8)
- moved U$1 0.30 mm to (14.3, 22.9)
- moved IC8 0.18 mm to (64.1, 21.1), turned to 0 degrees
- moved U$3 0.15 mm to (33.8, 48.3)
- moved U1 0.10 mm to (65.9, 42.5)
Connections:
- net HOME_SHUTTER_CLOSED renamed HOME_ROR_CLOSED
- net HOME_SHUTTER_CLOSED-IN_EXT renamed HOME_ROR_CLOSED-IN_EXT
- net HOME_SHUTTER_CLOSED_IN_5V renamed HOME_ROR_CLOSED_IN_5V
- net SHUTTER_OPENED renamed ROR_OPENED
- net SHUTTER_OPENED-IN_EXT renamed ROR_OPENED-IN_EXT
- net SHUTTER_OPENED_IN_5V renamed ROR_OPENED_IN_5V
- net 3.3V: now also R3.1; no longer C5.1, IC2.8, R1.2, R3.2
- net GND: now also R1.1; no longer C5.2, IC2.1, IC2.2, IC2.3, IC2.4
- net SCL: no longer IC2.6, R1.1
- net SDA: no longer IC2.5, R3.1
- net SPARE_OUT1: now also R3.2
- net SPARE_OUT2: now also R1.2
Routing:
- net SDA: track 16.4 -> 0.00 mm, vias 1 -> 0
- net SCL: track 11.5 -> 0.00 mm
- net 3.3V: track 158.6 -> 152.6 mm
- net SPARE_OUT2: track 39.5 -> 42.0 mm
- net SPARE_OUT1: track 12.5 -> 14.6 mm
- net AT_PARK_PIN_IN_5V: track 79.6 -> 78.3 mm
- net ROR_OPENED_IN_5V: track 48.9 -> 47.7 mm
- net HOME_ROR_CLOSED_IN_5V: track 56.5 -> 55.5 mm
- net SPARE2-IN_EXT: track 13.4 -> 14.4 mm
- net SPARE1_IN_5V: track 41.5 -> 40.5 mm
- net BUTTON_WEST_CLOSE_IN_5V: track 62.8 -> 61.8 mm
- net BUTTON_EAST_OPEN_5V: track 69.3 -> 68.3 mm
- net RG-11-IN_5V: track 41.2 -> 40.2 mm
- net SPARE2_IN_5V: track 30.4 -> 29.5 mm
Other:
- board text added: "Close RoR"
- board text added: "Close RoR / West"
- board text added: "Open RoR"
- board text added: "Open RoR / East"
- board text added: "RoR Closed"
- board text added: "RoR Closed / Home"
- board text added: "RoR Opened"
- board text removed: "Opened"
