File: Hardware/RTI-Dome-eth-ESP32/RTI-Dome-eth-ESP32.sch (EAGLE design)
At the start: 102 parts, among them IC2 24LC64T-I/SN, IC8 REG1117-3.3V, J1 691313510003, J10 691313510002, J11 691313510002, J12 691313510002, J2 XT60PW-M, J3 691313510003, J4 691313510003, J6 691313510003, J7 691313510003, J8 691313510002, J9 691313510002, T1 MMBT3904LT1, T2 MMBT3904LT1, T3 MMBT3904LT1, U1 W5500, U2 ESP32-DevKitC-32UE, X9 J1011F01PNL

Commit message: Adding latest PCB files
Parts:
- removed C5: 100nF, rcl:C-EUC0603
- removed IC2: 24LC64T-I/SN, rti:24LC64T-I/SN
- R1, R3: value 1K -> 100K; device rcl:R-EU_R0603 -> rti:R-EU'0603'; MPN RT0805FRE071KL -> RT0805FRD07100RL
- U$1: LCSC_PART (none) -> C131314
- U$3: LCSC_PART (none) -> C6093
Connections:
- net HOME_SHUTTER_CLOSED renamed HOME_ROR_CLOSED
- net HOME_SHUTTER_CLOSED-IN_EXT renamed HOME_ROR_CLOSED-IN_EXT
- net HOME_SHUTTER_CLOSED_IN_5V renamed HOME_ROR_CLOSED_IN_5V
- net SHUTTER_OPENED renamed ROR_OPENED
- net SHUTTER_OPENED-IN_EXT renamed ROR_OPENED-IN_EXT
- net SHUTTER_OPENED_IN_5V renamed ROR_OPENED_IN_5V
- net 3.3V: now also R3.1; no longer C5.1, IC2.VCC, R1.2, R3.2
- net GND: now also R1.1; no longer C5.2, IC2.A0, IC2.A1, IC2.A2, IC2.VSS
- net SCL: no longer IC2.SCL, R1.1
- net SDA: no longer IC2.SDA, R3.1
- net SPARE_OUT1: now also R3.2
- net SPARE_OUT2: now also R1.2
Other:
- moved on the sheet: C2, C27, R1, R3
